Commit message: updated CAD data and sysid

File: urdf/robot.urdf (robot description, URDF)
Before this commit: robot rotary_pendulum, 3 links, 2 joints
Links:
- link arm: mass 0.0341342 -> 0.0367867; geometry collision mesh filename=package://assets\608zz.stl; collision mesh filename=package://assets\composite_part_2.stl
- link base: mass 0.277405 -> 0.27687
- link pendulum: mass 0.00747898 -> 0.00903535
Joints:
- joint arm_to_pendulum: origin xyz=0.059 0 0.002 rpy=1.5708 0.0370451 1.5708 -> xyz=0.06 -0 0.002 rpy=1.5708 -0.00389442 1.5708; parent arm -> composite_part_2
- joint base_to_arm: child arm -> composite_part_2; origin xyz=-0 0.10295 -9.79797e-05 rpy=1.5708 1.5708 0 -> xyz=-0 0.0916803 0.0986761 rpy=3.14159 -0 -1.5708

Commit message: new sysid for FPGA

File: urdf/robot.urdf (robot description, URDF)
Before this commit: robot rotary_pendulum, 3 links, 2 joints
Joints:
- joint arm_to_pendulum: origin xyz=0.06 -0 0.002 rpy=1.5708 -0.00389442 1.5708 -> xyz=0.063 -0 0.002 rpy=1.5708 -0.00389442 1.5708
